Commit message: fix : no human rigging & actor mesh change

File: src/robot_control/urdf/mecanum_lift_robot.urdf.xacro (robot description, xacro)
@@ -10,11 +10,21 @@
 <robot name="mecanum_lift_robot" xmlns:xacro="http://www.ros.org/wiki/xacro">
   <xacro:arg name="ns" default="robot2"/>
-  <!-- ===== 외형 메시 (mecanum_lift) ===== -->
-  <!-- 원본 model.sdf의 visual pose(0 0 -0.084, roll 90도)를 그대로 재사용 —
-       이 메시는 원래부터 이 오프셋으로 정렬해서 쓰도록 만들어진 애셋이다. -->
-  <xacro:property name="lift_mesh" value="model://mecanum_lift/meshes/MecanumLift.dae"/>
-  <xacro:property name="lift_scale" value="0.6 0.6 0.6"/>
-  <xacro:property name="mesh_roll" value="1.5708"/>
-  <xacro:property name="mesh_z_offset" value="-0.084"/>
+  <!-- ===== 외형 메시 (deco_forklift 재사용) ===== -->
+  <!-- worlds/navi_factory 의 deco_forklift_ogv 소품과 같은 glb를 그대로 쓴다. 그 소품은
+       scale/offset 없이(즉 1:1 실척, 원점=바닥) 배치돼 있었으므로 여기서도 동일하게
+       회전·오프셋 없이 얹는다. 실제 지게차 실척(길이 2.4 x 폭 1.4 x 높이 2.06m)이라
+       지금 chassis collision(2.0x0.9x0.6)/바퀴 배치보다 눈에 띄게 크고 높다 — 요청은
+       "메시 교체"까지라 물리 치수(collision/wheel_sep 등)는 안 건드렸고, 시각적으로
+       안 맞으면 후속으로 chassis 치수도 지게차 실척에 맞춰 키우는 작업이 필요하다. -->
+  <xacro:property name="lift_mesh" value="model://Forklift/base_visual.glb"/>
+  <xacro:property name="lift_scale" value="1 1 1"/>
+  <xacro:property name="mesh_roll" value="0"/>
+  <xacro:property name="mesh_z_offset" value="0"/>
+  <!-- base_visual.glb 안에 Y축 +90도 회전이 이미 baked돼 있어(Blender glTF export 축변환
+       추정), 이 mesh_yaw 하나만으로는 정면이 로봇의 실제 전진(+X, DiffDrive/바퀴 기준)과
+       맞는다는 보장이 없다. Gazebo에서 정지 스폰해 포크가 향하는 쪽과 +X 전진 방향을
+       비교해 0/1.5708/3.1416/-1.5708 중 맞는 값으로 채워야 한다(로봇.urdf.xacro의
+       mesh_yaw 패턴과 동일). -->
+  <xacro:property name="mesh_yaw" value="0"/>
   <!-- ===== 구동 파라미터 ===== -->
   <xacro:property name="wheel_radius" value="0.15"/>
@@ -60,5 +70,5 @@
   <link name="chassis">
     <visual>
-      <origin xyz="0 0 ${mesh_z_offset}" rpy="${mesh_roll} 0 0"/>
+      <origin xyz="0 0 ${mesh_z_offset}" rpy="${mesh_roll} 0 ${mesh_yaw}"/>
       <geometry>
         <mesh filename="${lift_mesh}" scale="${lift_scale}"/>

Commit message: chore : yolo package import

File: src/robot_control/urdf/mecanum_lift_robot.urdf.xacro (robot description, xacro)
@@ -21,10 +21,10 @@
   <xacro:property name="mesh_roll" value="0"/>
   <xacro:property name="mesh_z_offset" value="0"/>
-  <!-- base_visual.glb 안에 Y축 +90도 회전이 이미 baked돼 있어(Blender glTF export 축변환
-       추정), 이 mesh_yaw 하나만으로는 정면이 로봇의 실제 전진(+X, DiffDrive/바퀴 기준)과
-       맞는다는 보장이 없다. Gazebo에서 정지 스폰해 포크가 향하는 쪽과 +X 전진 방향을
-       비교해 0/1.5708/3.1416/-1.5708 중 맞는 값으로 채워야 한다(로봇.urdf.xacro의
-       mesh_yaw 패턴과 동일). -->
-  <xacro:property name="mesh_yaw" value="0"/>
+  <!-- base_visual.glb 안에 Y축 +90도 회전이 이미 baked돼 있다(glTF 노드 rotation
+       [0, 0.7071, 0, 0.7071] 확인됨). 노드 rotation+scale을 반영해 정점을 직접
+       변환해보면 mesh_yaw=0일 때 포크(바닥 근처 저-z 밴드가 몸통보다 튀어나온 방향)가
+       로컬 +Y를 향한다 — 로봇 전진(+X, DiffDrive)과 90도 어긋난다. -1.5708(-90도)을
+       주면 포크가 +X를 향하도록 검증했다. -->
+  <xacro:property name="mesh_yaw" value="-1.5708"/>
   <!-- ===== 구동 파라미터 ===== -->
   <xacro:property name="wheel_radius" value="0.15"/>

Commit message: fixed :  human patrol feat :  view division fix : auto - drive

File: src/robot_control/urdf/mecanum_lift_robot.urdf.xacro (robot description, xacro)
@@ -99,4 +99,22 @@
             </ode>
           </friction>
+          <!-- '스톨' 버그(바퀴 관절은 명령대로 도는데 차체가 접지력을 못 받고
+               멈추는 현상) 원인 재분석: 바퀴 바닥(-0.01, chassis 원점 기준)과
+               캐스터 바닥(+0.02, 아래 캐스터 매크로 참고)이 3cm나 어긋나 있어서,
+               평상시 순항 중엔 캐스터가 바닥에서 3cm 떠 있다가 급가감속으로
+               섀시가 피치(앞뒤 기울임)할 때만 갑자기 캐스터가 바닥에 부딪히듯
+               접촉하게 되는 구조였다 — 이런 "상대속도가 있는 상태에서 갑자기
+               새로 생기는 접촉"이 DART 접촉 솔버에 불안정한 입력이 되어 접촉력을
+               잘못 계산(0으로 반환)하는 것으로 보인다. contact_max_correcting_vel/
+               min_depth를 낮춰 침투 보정을 부드럽게 하고, kp/kd로 접촉 강성 자체를
+               유한하게(무한강성 아니게) 줘서 순간적인 충격성 접촉이 생겨도 힘이
+               한 스텝에 몰리지 않게 한다. -->
+          <contact>
+            <ode>
+              <min_depth>0.001</min_depth>
+              <kp>1e6</kp>
+              <kd>100</kd>
+            </ode>
+          </contact>
         </surface>
       </collision>
@@ -112,4 +130,9 @@
   <xacro:drive_wheel prefix="right" side_y="${-wheel_sep/2}"/>
   <!-- ===== 캐스터 매크로 (앞/뒤 지지, 마찰 0) ===== -->
+  <!-- 바퀴와 같은 방식(반지름-0.01)으로 바닥에서 같은 깊이만큼 파묻히게 맞춰서,
+       스폰 직후 중력으로 가라앉아 자리잡을 때 바퀴/캐스터 4점이 동시에 자리를
+       잡는다 — 예전엔 캐스터 바닥이 바퀴보다 3cm 높아서 평상시엔 안 닿다가
+       급가감속으로 섀시가 기울 때만 갑자기 닿는 구조였고, 그 순간접촉이 스톨의
+       원인으로 보였다(위 wheel contact 주석 참고). -->
   <xacro:macro name="caster" params="prefix px">
     <link name="${prefix}_caster">
@@ -122,8 +145,24 @@
       <parent link="chassis"/>
       <child  link="${prefix}_caster"/>
-      <origin xyz="${px} 0 ${caster_radius + 0.02}" rpy="0 0 0"/>
+      <origin xyz="${px} 0 ${caster_radius - 0.01}" rpy="0 0 0"/>
     </joint>
     <gazebo reference="${prefix}_caster">
-      <mu1>0.0</mu1><mu2>0.0</mu2>
+      <collision>
+        <surface>
+          <friction>
+            <ode>
+              <mu>0.0</mu>
+              <mu2>0.0</mu2>
+            </ode>
+          </friction>
+          <contact>
+            <ode>
+              <min_depth>0.001</min_depth>
+              <kp>1e6</kp>
+              <kd>100</kd>
+            </ode>
+          </contact>
+        </surface>
+      </collision>
     </gazebo>
   </xacro:macro>
