Commit message: feature: knavi_robot 에 2D 라이다 추가하고 센서 frame_id 를 고정
robot.urdf.xacro 에 lidar_link 와 gpu_lidar 센서를 달고 bridge.yaml 에
/robot1/scan 을 추가한다. 마운트 높이 0.65 m 는 차체 collision 박스
(z=0.15~0.55)보다 위여야 360° 스캔이 자기 몸통에 막히지 않기 때문이고,
min range 0.3 도 자기 반사를 배제하려는 같은 이유다.

센서 토픽에 gz_frame_id 를 명시한다 — 없으면 ROS 로 넘어온 LaserScan/Image
의 frame_id 가 "knavi_robot/lidar_link/lidar" 같은 gz 내부 스코프 이름이
되어 Nav2 의 tf 조회가 실패한다.

Co-Authored-By: Claude Opus 5 <noreply@anthropic.com>

File: src/robot_control/urdf/mecanum_lift_robot.urdf.xacro (robot description, xacro)
@@ -182,4 +182,8 @@
            camera/image로 전역 토픽이라 로봇이 여러 대면 충돌할 뻔했다. -->
       <topic>$(arg ns)/camera/image</topic>
+      <!-- gz_frame_id 를 반드시 넣는다: 없으면 ROS 로 넘어온 Image 의 frame_id 가
+           "mecanum_lift_robot/camera_link/sim_camera" 같은 gz 내부 스코프 이름이 되어
+           tf 조회(카메라 좌표 → base_link)가 실패한다. -->
+      <gz_frame_id>camera_link</gz_frame_id>
       <camera>
         <horizontal_fov>1.047</horizontal_fov>
@@ -196,4 +200,7 @@
     <sensor name="lidar" type="gpu_lidar">
       <topic>$(arg ns)/scan</topic>
+      <!-- 카메라와 같은 이유. 없으면 LaserScan 의 frame_id 가 gz 내부 스코프 이름이 되어
+           Nav2 가 tf 조회에 실패한다. -->
+      <gz_frame_id>lidar_link</gz_frame_id>
       <update_rate>5</update_rate>
       <lidar>

File: src/robot_control/urdf/robot.urdf.xacro (robot description, xacro)
@@ -149,4 +149,17 @@
     <origin xyz="0.5 0 0.5" rpy="0 0 0"/>
   </joint>
+  <!-- ===== 2D LiDAR 링크 (Nav2 입력: SLAM·AMCL·costmap 전부 이 스캔을 쓴다) =====
+       마운트 높이 0.65 m 의 근거: 차체 collision 박스가 z=0.15~0.55 라, 그보다 위여야
+       360° 스캔이 자기 몸통에 막히지 않는다. min range 0.3 도 같은 이유(자기 반사 배제).
+       한계: 2D 라이다는 이 높이의 수평 단면 한 장만 본다. 바닥의 팔레트처럼 낮은 물체,
+       머리 위로 튀어나온 물체는 안 잡힌다. 3D 커버는 나중에 깊이 카메라(voxel layer)로 보강. -->
+  <link name="lidar_link">
+    <xacro:box_inertia m="0.1" x="0.06" y="0.06" z="0.06"/>
+  </link>
+  <joint name="lidar_joint" type="fixed">
+    <parent link="base_link"/>
+    <child  link="lidar_link"/>
+    <origin xyz="0 0 0.65" rpy="0 0 0"/>
+  </joint>
   <!-- ================= Gazebo (gz-sim / Harmonic) ================= -->
   <gazebo>
@@ -173,5 +186,7 @@
       <always_on>1</always_on>
       <update_rate>15</update_rate>
-      <topic>camera/image</topic>
+      <!-- ns 를 붙여 로봇이 여러 대여도 토픽이 안 겹치게. bridge.yaml 과 이름이 일치해야 한다. -->
+      <topic>$(arg ns)/camera/image</topic>
+      <gz_frame_id>camera_link</gz_frame_id>
       <camera>
         <horizontal_fov>1.047</horizontal_fov>
@@ -181,3 +196,35 @@
     </sensor>
   </gazebo>
+  <!-- LiDAR 센서 정의.
+       gz_frame_id 를 반드시 넣는다: 없으면 ROS 로 넘어온 LaserScan 의 frame_id 가
+       "knavi_robot/lidar_link/lidar" 같은 gz 내부 스코프 이름이 되어, Nav2 가 tf 조회에 실패한다. -->
+  <gazebo reference="lidar_link">
+    <sensor name="lidar" type="gpu_lidar">
+      <always_on>1</always_on>
+      <update_rate>10</update_rate>
+      <visualize>true</visualize>
+      <topic>$(arg ns)/scan</topic>
+      <gz_frame_id>lidar_link</gz_frame_id>
+      <lidar>
+        <scan>
+          <horizontal>
+            <samples>720</samples>          <!-- 360°/720 = 0.5° 해상도 -->
+            <resolution>1</resolution>
+            <min_angle>-3.14159</min_angle>
+            <max_angle>3.14159</max_angle>
+          </horizontal>
+        </scan>
+        <range>
+          <min>0.3</min>                    <!-- 차체 자기 반사 배제 -->
+          <max>20.0</max>                   <!-- slam_toolbox max_laser_range 와 맞춤 -->
+          <resolution>0.01</resolution>
+        </range>
+        <noise>
+          <type>gaussian</type>
+          <mean>0.0</mean>
+          <stddev>0.01</stddev>
+        </noise>
+      </lidar>
+    </sensor>
+  </gazebo>
 </robot>

Commit message: fixed: 라이다를 몸통 안에서 앞 범퍼로 옮김
라이다가 창고를 전혀 못 보고 있었다. chassis 기준 (0.3, 0, 1.1) 은 mecanum_lift
외형 메시 "안쪽"이라, 광선 360개가 전부 0.32~1.43m 에서 자기 몸에 맞았다.
gpu_lidar 는 collision 이 아니라 visual 을 렌더링해서 맞히기 때문에, URDF
collision 박스(높이 0.6)를 넘긴 것만으로는 소용이 없었다.

확인 방법: 바닥판을 끈 실행에서 로봇이 결함 STL 바닥을 뚫고 z=-241m 로 떨어져
있었는데, 바닥판을 켜 z=0.23m 에 정상히 세운 실행과 스캔이 각도별 값까지
동일했다. 지하 241m 허공에서도 같은 게 보인다면 그건 로봇을 따라다니는 물체다.
MecanumLift.dae 를 COLLADA 씬 그래프(단위 0.01m, Y_UP)까지 반영해 재면 chassis
기준 bbox 가 x[-1.07,0.99] y[-0.61,0.34] z[0.08,2.01] 이고, 각 면까지의 계산
거리(앞 0.69 / 뒤 1.37 / 좌 0.34 / 우 0.61)가 실측 스캔과 2cm 안에서 맞는다.

그 footprint 가 높이 0~2.01m 전 구간에서 유지되어 몸통 안에는 트이는 높이가
없다. 위(z>2.01)로 올리면 2.15m 수평 단면이라 사람도 팔레트도 그 아래로
지나가므로, 신호수 안전이 목적인 이 프로젝트에는 맞지 않는다. 그래서 앞으로
뺐다: x=1.05 는 메시 앞면(0.988)과 collision 박스 앞면(1.0) 둘 다 바깥이고,
z=0.5 는 사람 다리와 팔레트가 걸리는 높이다.

옮긴 뒤 실측: 최대 9.61m 까지 창고 구조물이 보인다. 다만 뒤쪽은 여전히 몸통에
막혀 광선 164/360개(46%)가 자기 자신에 맞고, 트인 구간은 -95.8도 ~ +99.8도다.
시야각을 그 구간으로 좁힐지는 아직 결정하지 않았다(doc/design.md 참고).

Co-Authored-By: Claude Opus 5 <noreply@anthropic.com>

File: src/robot_control/urdf/mecanum_lift_robot.urdf.xacro (robot description, xacro)
@@ -130,4 +130,15 @@
   </joint>
   <!-- ===== 라이다 링크 ===== -->
+  <!-- 앞 범퍼 위치. 예전엔 (0.3, 0, 1.1) 이었는데 그건 외형 메시 "안쪽"이라
+       360개 광선이 전부 0.32~1.43m 에서 자기 몸에 맞았다(창고 벽은 하나도 안 보였음).
+       collision 박스(높이 0.6)는 넘겼지만 gpu_lidar 는 collision 이 아니라 visual 을
+       렌더링해서 맞히기 때문에 소용이 없었다.
+       MecanumLift.dae 를 COLLADA 씬 그래프(단위 0.01m, Y_UP)까지 반영해 재 보면
+       chassis 기준 bbox 가 x[-1.07,0.99] y[-0.61,0.34] z[0.08,2.01] 이고, 그 footprint 가
+       높이 0~2.01m 전 구간에서 유지된다 — 몸통 안에는 트이는 높이가 없다.
+       위(z>2.01)로 올리는 방법도 있지만 2.15m 수평 단면은 사람도 팔레트도 그 아래로
+       지나가서, 신호수 안전이 목적인 이 프로젝트에는 맞지 않는다. 그래서 앞으로 뺐다:
+       x=1.05 는 메시 앞면(0.988)과 collision 박스 앞면(1.0) 둘 다 바깥이고,
+       z=0.5 는 사람 다리·팔레트·콘이 걸리는 높이다. -->
   <link name="lidar_link">
     <xacro:box_inertia m="0.1" x="0.05" y="0.05" z="0.05"/>
@@ -136,5 +147,5 @@
     <parent link="chassis"/>
     <child  link="lidar_link"/>
-    <origin xyz="0.3 0 1.1" rpy="0 0 0"/>
+    <origin xyz="1.05 0 0.5" rpy="0 0 0"/>
   </joint>
   <!-- ================= Gazebo (gz-sim / Harmonic) ================= -->

Commit message: fixed: 차체 물리 치수를 지게차 메시 실측에 맞추고 라이다를 앞 범퍼로 옮김
외형 메시가 MecanumLift 에서 Forklift 로 바뀌었는데 물리 치수는 옛 값
(2.0x0.9x0.6, wheel_sep 1.3, caster_x 0.95)이 그대로 남아 근거가 사라진
상태였다. 계산으로 glTF 좌표를 변환해 보려 했지만 두 번 다 실측과 안 맞아서
(Y-up 변환 가정 문제) 시뮬레이션에서 직접 쟀다 — 라이다를 차체 밖 6m 지점
(정면 x=+6, 측면 y=+6)에 두고 자기 몸을 스캔해 높이별 실루엣을 읽는 방식이다.

  높이 0.3m : x[-0.85, 1.10]  y[-0.52, 0.57]
  높이 0.6m : x[-0.80, 1.10]  y[-0.52, 0.55]
  높이 1.5m : x[-0.67, 0.96]  y[-0.48, 0.49]
  위끝      : z=2.1m 에는 반사 있고 z=2.3m 에는 없음
  => 길이 1.95, 폭 1.09, 높이 약 2.2, 중심이 x=+0.125

월드 소품 deco_forklift_ogv 의 collision box 에 적힌 2.4x1.4x2.06 은 이 메시의
실제 크기가 아니다. 그 값을 믿고 맞추면 안 된다.

바뀐 것:
- collision box 2.0x0.9x0.6 @z=0.45 -> 1.95x1.09x2.05 @(0.125, 0, 1.175).
  바닥에서 0.15m 띄운다 — 0 이면 박스가 먼저 닿아 바퀴가 뜨고 안 굴러간다.
- wheel_sep 1.3 -> 0.95. 옛 값은 차체 폭 0.9 기준이라 지금 메시에서 바퀴가
  좌우로 0.17m 씩 삐져나왔다.
- caster_x 0.95 -> 0.72. 뒤 캐스터가 차체 뒤끝(-0.85) 밖 허공에 떠 있었다.
- 라이다 (1.05, 0, 0.50) -> (1.25, 0, 0.35). 후보를 한 실행에서 동시에 재서
  골랐다: 이전 값 57% 막힘/±75.7도, 이 값 41%/±105.8도, 마스트 위(0.125,0,2.40)
  0%/완전 360도. 마스트 위는 지면 2.4m 단면이라 사람도 팔레트도 그 아래로
  지나가서 안전 목적에 못 쓴다 — 실물 AGV 도 항법용은 마스트 위, 안전용은 낮게
  따로 단다. z=0.35 는 사람 다리와 팔레트가 걸리는 높이다.

collision 높이를 0.6 에서 2.05 로 키우면 선반에 걸릴 수 있어 patrol 로 확인했다:
30초에 15.52m, 10초 구간 5개 모두 정상(9.39/4.10/10.63/8.30/1.80m),
roll·pitch 1도 이내, z 0.22~0.24 유지.

base_mass 는 25kg 그대로 뒀다. 지게차 실척이면 수천 kg 인데 그건 치수가 아니라
동역학이 통째로 바뀌는 변경이라 따로 결정할 일이다.

Co-Authored-By: Claude Opus 5 <noreply@anthropic.com>

File: src/robot_control/urdf/mecanum_lift_robot.urdf.xacro (robot description, xacro)
@@ -27,11 +27,37 @@
        주면 포크가 +X를 향하도록 검증했다. -->
   <xacro:property name="mesh_yaw" value="-1.5708"/>
+  <!-- ===== 차체 실측 치수 =====
+       외형 메시를 지게차로 바꾸면서 물리 치수는 옛 값(2.0x0.9x0.6)이 남아 있었다.
+       그 값들의 근거가 사라졌으므로 실제 렌더되는 메시를 시뮬레이션에서 직접 쟀다:
+       라이다를 차체 밖 6m 지점(정면 x=+6, 측면 y=+6)에 두고 자기 몸을 스캔해
+       높이별 실루엣을 읽는 방식이다. 계산으로 glTF 좌표를 변환해 보기도 했는데
+       두 번 다 실측과 안 맞아서(Y-up 변환 가정 문제) 계산값은 쓰지 않았다.
+         높이 0.3m : x[-0.85, 1.10]  y[-0.52, 0.57]
+         높이 0.6m : x[-0.80, 1.10]  y[-0.52, 0.55]
+         높이 1.5m : x[-0.67, 0.96]  y[-0.48, 0.49]
+         위끝      : z=2.1m 에는 반사 있고 z=2.3m 에는 없음
+       => 길이 1.95, 폭 1.09, 높이 약 2.2. 앞뒤로는 원점 기준 앞이 더 길다
+       (중심이 x=+0.125). 월드 소품 deco_forklift_ogv 의 collision box 에 적힌
+       2.4x1.4x2.06 은 이 메시의 실제 크기가 아니다 — 그 값을 믿고 맞추면 안 된다. -->
+  <xacro:property name="body_len"    value="1.95"/>
+  <xacro:property name="body_wid"    value="1.09"/>
+  <xacro:property name="body_x"      value="0.125"/>  <!-- 차체 중심의 x 오프셋 -->
+  <xacro:property name="body_top"    value="2.2"/>
+  <!-- 지면과 차체 바닥 사이 간격. 0 으로 두면 collision 박스가 바닥에 먼저 닿아
+       바퀴가 뜨고 로봇이 굴러가지 않는다. -->
+  <xacro:property name="ground_gap"  value="0.15"/>
   <!-- ===== 구동 파라미터 ===== -->
   <xacro:property name="wheel_radius" value="0.15"/>
   <xacro:property name="wheel_width"  value="0.12"/>
-  <!-- 고속 코너링 시 전복 방지: 바퀴/캐스터 간격을 넓혀 안정성 확보 -->
-  <xacro:property name="wheel_sep"    value="1.3"/>
+  <!-- 바퀴가 차체 폭(1.09) 밖으로 튀어나오지 않게 잡는다: 1.3 이던 예전 값은
+       옛 차체(폭 0.9) 기준이라 지금 메시에서는 바퀴가 좌우로 0.17m 씩 삐져나왔다.
+       0.95 면 바깥면이 0.95/2+0.12/2 = 0.535 로 차체 반폭 0.545 안에 들어온다.
+       전복 걱정은 이 모델에선 크지 않다 — box_inertia 매크로가 <origin> 을 주지
+       않아 무게중심이 링크 원점(지면 높이)에 있기 때문이다. -->
+  <xacro:property name="wheel_sep"    value="0.95"/>
   <xacro:property name="caster_radius" value="0.07"/>
-  <xacro:property name="caster_x"      value="0.95"/>
+  <!-- 캐스터도 차체 안쪽으로. 0.95 였을 때 뒤 캐스터(-0.95)가 차체 뒤끝(-0.85)
+       밖으로 나가 허공에 떠 있었다. 앞뒤 짧은 쪽(0.85)에서 여유를 둔 값이다. -->
+  <xacro:property name="caster_x"      value="0.72"/>
   <xacro:property name="base_mass"   value="25.0"/>
   <xacro:property name="wheel_mass"  value="1.5"/>
@@ -75,9 +101,13 @@
       </geometry>
     </visual>
+    <!-- collision 박스를 실측 치수로. 바닥에서 ground_gap 만큼 띄우고 body_top 까지
+         올린다 — 위끝을 2.2 로 잡으면 지게차 마스트까지 포함되므로, 로봇이 선반
+         아래를 통과하던 게 이제 막힐 수 있다(예전 박스는 높이 0.6 뿐이었다). -->
+    <xacro:property name="body_hgt" value="${body_top - ground_gap}"/>
     <collision>
-      <origin xyz="0 0 0.45" rpy="0 0 0"/>
-      <geometry><box size="2.0 0.9 0.6"/></geometry>
+      <origin xyz="${body_x} 0 ${ground_gap + body_hgt/2}" rpy="0 0 0"/>
+      <geometry><box size="${body_len} ${body_wid} ${body_hgt}"/></geometry>
     </collision>
-    <xacro:box_inertia m="${base_mass}" x="2.0" y="0.9" z="0.6"/>
+    <xacro:box_inertia m="${base_mass}" x="${body_len}" y="${body_wid}" z="${body_hgt}"/>
   </link>
   <!-- ===== 구동 바퀴 매크로 ===== -->
@@ -140,15 +170,18 @@
   </joint>
   <!-- ===== 라이다 링크 ===== -->
-  <!-- 앞 범퍼 위치. 예전엔 (0.3, 0, 1.1) 이었는데 그건 외형 메시 "안쪽"이라
-       360개 광선이 전부 0.32~1.43m 에서 자기 몸에 맞았다(창고 벽은 하나도 안 보였음).
-       collision 박스(높이 0.6)는 넘겼지만 gpu_lidar 는 collision 이 아니라 visual 을
-       렌더링해서 맞히기 때문에 소용이 없었다.
-       MecanumLift.dae 를 COLLADA 씬 그래프(단위 0.01m, Y_UP)까지 반영해 재 보면
-       chassis 기준 bbox 가 x[-1.07,0.99] y[-0.61,0.34] z[0.08,2.01] 이고, 그 footprint 가
-       높이 0~2.01m 전 구간에서 유지된다 — 몸통 안에는 트이는 높이가 없다.
-       위(z>2.01)로 올리는 방법도 있지만 2.15m 수평 단면은 사람도 팔레트도 그 아래로
-       지나가서, 신호수 안전이 목적인 이 프로젝트에는 맞지 않는다. 그래서 앞으로 뺐다:
-       x=1.05 는 메시 앞면(0.988)과 collision 박스 앞면(1.0) 둘 다 바깥이고,
-       z=0.5 는 사람 다리·팔레트·콘이 걸리는 높이다. -->
+  <!-- 앞 범퍼, 다리 높이. gpu_lidar 는 collision 이 아니라 visual 을 렌더링해서
+       맞히므로, collision 박스를 피하는 것만으로는 자기 몸을 안 보게 할 수 없다.
+       위치를 시뮬레이션에서 후보별로 재 봤다(막힌 광선 비율 / 연속으로 트인 각):
+         (1.05, 0, 0.50) 이전 값   57% 막힘   ±75.7도
+         (1.25, 0, 0.35) 이 값     41% 막힘   ±105.8도
+         (1.25, 0, 0.60)           41% 막힘   ±105.8도
+         (0.125, 0, 2.40) 마스트 위 0% 막힘   완전 360도
+       마스트 위가 유일하게 진짜 360도지만, 지면 2.4m 높이의 수평 단면이라 사람도
+       팔레트도 콘도 그 아래로 지나간다. 신호수 안전이 목적인 1단계에는 못 쓴다.
+       실물 AGV 도 항법용 라이다는 마스트 위, 안전용 스캐너는 낮게 따로 단다.
+       그래서 안전용 쪽을 골랐다: x=1.25 는 차체 앞끝(1.10) 바로 앞이고,
+       z=0.35 는 사람 다리와 팔레트가 걸리는 높이다.
+       뒤쪽 41% 는 차체에 막힌 채로 남는다 — 뒤를 보려면 뒤 범퍼에 한 대를 더
+       달아야 하고(실물 AGV 의 대각선 2대 배치), 지금은 후진을 안 하므로 미룬다. -->
   <link name="lidar_link">
     <xacro:box_inertia m="0.1" x="0.05" y="0.05" z="0.05"/>
@@ -157,5 +190,5 @@
     <parent link="chassis"/>
     <child  link="lidar_link"/>
-    <origin xyz="1.05 0 0.5" rpy="0 0 0"/>
+    <origin xyz="1.25 0 0.35" rpy="0 0 0"/>
   </joint>
   <!-- ================= Gazebo (gz-sim / Harmonic) ================= -->

Commit message: fixed: 차체가 바닥판을 관통해 끼는 문제와 무게중심 위치
주행 중 로봇이 코를 든 채 그 자리에 박혀 바퀴만 헛도는 현상이 반복됐다.
살아 있는 시뮬에서 잰 값:

  바퀴 각속도 20.4 / 23.0 rad/s (림 3.1m/s)  실제 이동 12초에 1cm
  피치 -18~19도 고정, 구동 토크를 6초간 끊어도 자세가 안 풀림

토크를 끊어도 안 풀린다는 건 동역학이 아니라 기하학적으로 끼었다는 뜻이다.
그 자세(원점 z=0.254, 피치 18.3도)에 URDF 치수를 넣으면 차체 박스 뒤아래
모서리가 z=0.13 — 두께 0.1m 짜리 바닥판(0.15~0.25) 아래로 2cm 빠져나가 있다.
빠른 속도로 크게 기울면 물리 스텝 한 번에 관통해 버린 것이다.

두 가지를 고친다:
- flat_ground 두께 0.1m → 4m. pose 를 반두께만큼 내려 윗면 높이(0.25)는 그대로
  유지하므로 주행 높이·스폰 위치는 안 바뀐다. static 박스라 비용도 없고, 월드
  모델 196개가 전부 static 이라 판 안에 묻히는 소품과는 접촉 계산 자체가 없다.
- 무게중심을 x=0.0067 → 0.125(차체 기하 중심), z=0.3 으로. 예전에는 box_inertia
  가 <origin> 을 안 줘서 무게중심이 구동축(x=0) 바로 위에 얹혀 있었고, 뒤로
  젖히는 토크를 되돌리는 모멘트가 1.8 N.m 뿐이었다 — 가속에 필요한 바퀴 토크
  5.9 N.m 보다 작아서 정상 가속만으로도 넘어갈 수 있는 상태였다. 32 N.m 가 된다.

Co-Authored-By: Claude Opus 5 <noreply@anthropic.com>

File: src/robot_control/urdf/mecanum_lift_robot.urdf.xacro (robot description, xacro)
@@ -53,6 +53,7 @@
        옛 차체(폭 0.9) 기준이라 지금 메시에서는 바퀴가 좌우로 0.17m 씩 삐져나왔다.
        0.95 면 바깥면이 0.95/2+0.12/2 = 0.535 로 차체 반폭 0.545 안에 들어온다.
-       전복 걱정은 이 모델에선 크지 않다 — box_inertia 매크로가 <origin> 을 주지
-       않아 무게중심이 링크 원점(지면 높이)에 있기 때문이다. -->
+       무게중심을 z=0.3 으로 올린 뒤의 좌우 전복 여유: 바퀴 반간격 0.475 기준으로
+       횡가속 9.81 x 0.475 / 0.3 = 15.5 m/s^2 까지 버틴다. 순항 3.33m/s 에서 이
+       값에 닿으려면 회전 반경이 0.7m 여야 하므로 트랙 주행에서는 문제되지 않는다. -->
   <xacro:property name="wheel_sep"    value="0.95"/>
   <xacro:property name="caster_radius" value="0.07"/>
@@ -63,6 +64,10 @@
   <xacro:property name="wheel_mass"  value="1.5"/>
   <!-- ===== 관성 매크로 ===== -->
-  <xacro:macro name="box_inertia" params="m x y z">
+  <!-- px/py/pz 는 무게중심 위치(링크 원점 기준). 기본 0 이라 이 값을 안 주면
+       예전처럼 무게중심이 링크 원점에 놓인다. 관성 텐서는 박스 중심 기준 값이므로
+       그 중심을 어디에 둘지를 여기서 정하는 셈이다. -->
+  <xacro:macro name="box_inertia" params="m x y z px:=0 py:=0 pz:=0">
     <inertial>
+      <origin xyz="${px} ${py} ${pz}" rpy="0 0 0"/>
       <mass value="${m}"/>
       <inertia ixx="${m*(y*y+z*z)/12.0}" ixy="0" ixz="0"
@@ -109,5 +114,16 @@
       <geometry><box size="${body_len} ${body_wid} ${body_hgt}"/></geometry>
     </collision>
-    <xacro:box_inertia m="${base_mass}" x="${body_len}" y="${body_wid}" z="${body_hgt}"/>
+    <!-- 무게중심을 차체 기하 중심의 x(=0.125)로 옮긴다. 예전에는 <origin> 이 없어
+         무게중심이 링크 원점, 즉 구동축(x=0) 바로 위에 얹혀 있었다 — 뒤로 넘어가려는
+         토크를 되돌리는 모멘트가 26.15kg x 9.81 x 0.0067m = 1.8 N.m 뿐이었다.
+         가속 1.5m/s^2 을 내려면 바퀴에 26.15 x 1.5 x 0.15 = 5.9 N.m 이 필요하고 그
+         반작용이 그대로 차체를 젖히므로, 복원 모멘트가 그보다 작으면 뒤집힌다.
+         x=0.125 면 복원 모멘트가 32 N.m 로 반작용의 5배가 넘는다.
+         z 는 0.3 으로 낮게 둔다: 실제 지게차도 배터리·카운터웨이트가 바닥에 있고,
+         높이면 (a) 코너에서 전복 여유가 줄고 (b) 가속 관성력의 팔 길이가 늘어
+         앞들림이 다시 심해진다(z=0.6 이면 젖히는 모멘트가 29 N.m 로 복원 32 N.m 에
+         육박한다). 관성 텐서 자체는 박스 전체 치수 기준 값을 그대로 쓴다. -->
+    <xacro:box_inertia m="${base_mass}" x="${body_len}" y="${body_wid}" z="${body_hgt}"
+                       px="${body_x}" pz="0.3"/>
   </link>
   <!-- ===== 구동 바퀴 매크로 ===== -->

Commit message: fixed: 바퀴 collision을 원통에서 구로 교체 — bullet 검출기의 원통-박스 접촉 불안정 회피
Co-Authored-By: Claude Fable 5 <noreply@anthropic.com>

File: src/robot_control/urdf/mecanum_lift_robot.urdf.xacro (robot description, xacro)
@@ -130,7 +130,12 @@
   <xacro:macro name="drive_wheel" params="prefix side_y">
     <link name="${prefix}_wheel">
+      <!-- collision 을 원통이 아니라 구(sphere)로 둔다. bullet 충돌 검출기는
+           원통-박스(바퀴-flat_ground) 접촉의 접촉점 생성이 불안정해서, 정지
+           상태에서 접촉력이 0 으로 풀리는 스톨(명령을 줘도 수 분간 출발/제자리
+           회전 불가, 2026-08-02 실측 287초)이 났다. 구는 어느 검출기에서도 접촉이
+           바닥 중앙 1점으로 유일하게 잡힌다. 반지름이 같아 차체 높이는 그대로고,
+           바닥이 평평한 이 월드(flat_ground)에서는 굴림 기하도 원통과 동일하다. -->
       <collision>
-        <origin xyz="0 0 0" rpy="1.5708 0 0"/>
-        <geometry><cylinder radius="${wheel_radius}" length="${wheel_width}"/></geometry>
+        <geometry><sphere radius="${wheel_radius}"/></geometry>
       </collision>
       <xacro:cyl_inertia m="${wheel_mass}" r="${wheel_radius}" l="${wheel_width}"/>
